Commit message: 更新 PUMA 机械臂的 URDF 模型，添加连杆和关节定义，优化可视化材料，包含任务目标文档

File: src/midterm_model/urdf/robot.urdf.xacro (robot description, xacro)
@@ -1,5 +1,28 @@
 <?xml version="1.0" ?>
-<robot name="robot1" xmlns:xacro="http://www.ros.org/wiki/xacro">
-<!-- Dummy root for KDL-->
+<robot name="puma_robot" xmlns:xacro="http://www.ros.org/wiki/xacro">
+    <!-- ============================================== -->
+    <!-- Material Definitions for Visualization        -->
+    <!-- ============================================== -->
+    <material name="blue">
+        <color rgba="0.0 0.0 0.8 1.0"/>
+    </material>
+    <material name="green">
+        <color rgba="0.0 0.8 0.0 1.0"/>
+    </material>
+    <material name="red">
+        <color rgba="0.8 0.0 0.0 1.0"/>
+    </material>
+    <material name="orange">
+        <color rgba="1.0 0.5 0.0 1.0"/>
+    </material>
+    <material name="yellow">
+        <color rgba="1.0 1.0 0.0 1.0"/>
+    </material>
+    <material name="grey">
+        <color rgba="0.5 0.5 0.5 1.0"/>
+    </material>
+    <!-- ============================================== -->
+    <!-- Dummy root for KDL                            -->
+    <!-- ============================================== -->
     <link name="dummy_root"/>
     <joint name="basejoint" type="fixed">
@@ -8,6 +31,193 @@
         <origin xyz="0 0 0" rpy="0 0 0"/>
     </joint>
-<!--END of Dummy root-->
-<!-- Start of robot description -->
-<!-- End of robot description -->
+    <!-- ============================================== -->
+    <!-- Link: base_link (基座)                         -->
+    <!-- Cylinder: radius=0.35, length=0.1             -->
+    <!-- ============================================== -->
+    <link name="base_link">
+        <visual>
+            <origin xyz="0 0 0.05" rpy="0 0 0"/>
+            <geometry>
+                <cylinder radius="0.35" length="0.1"/>
+            </geometry>
+            <material name="grey"/>
+        </visual>
+        <collision>
+            <origin xyz="0 0 0.05" rpy="0 0 0"/>
+            <geometry>
+                <cylinder radius="0.35" length="0.1"/>
+            </geometry>
+        </collision>
+        <inertial>
+            <mass value="10.0"/>
+            <origin xyz="0 0 0.05" rpy="0 0 0"/>
+            <inertia ixx="1.0" ixy="0.0" ixz="0.0" iyy="1.0" iyz="0.0" izz="1.0"/>
+        </inertial>
+    </link>
+    <!-- ============================================== -->
+    <!-- Joint: J_0 (Revolute)                         -->
+    <!-- Connects base_link to link_01                 -->
+    <!-- Origin: xyz="0 0 0.1", Axis: Z                -->
+    <!-- ============================================== -->
+    <joint name="J_0" type="revolute">
+        <parent link="base_link"/>
+        <child link="link_01"/>
+        <origin xyz="0 0 0.1" rpy="0 0 0"/>
+        <axis xyz="0 0 1"/>
+        <limit lower="-3.14" upper="3.14" effort="100" velocity="1.0"/>
+    </joint>
+    <!-- ============================================== -->
+    <!-- Link: link_01 (第一臂/立柱)                    -->
+    <!-- Cylinder: radius=0.15, length=1.1             -->
+    <!-- ============================================== -->
+    <link name="link_01">
+        <visual>
+            <origin xyz="0 0 0.55" rpy="0 0 0"/>
+            <geometry>
+                <cylinder radius="0.15" length="1.1"/>
+            </geometry>
+            <material name="blue"/>
+        </visual>
+        <collision>
+            <origin xyz="0 0 0.55" rpy="0 0 0"/>
+            <geometry>
+                <cylinder radius="0.15" length="1.1"/>
+            </geometry>
+        </collision>
+        <inertial>
+            <mass value="5.0"/>
+            <origin xyz="0 0 0.55" rpy="0 0 0"/>
+            <inertia ixx="0.5" ixy="0.0" ixz="0.0" iyy="0.5" iyz="0.0" izz="0.5"/>
+        </inertial>
+    </link>
+    <!-- ============================================== -->
+    <!-- Joint: J_F0 (Fixed) - 坐标系转换关节           -->
+    <!-- Connects link_01 to link_01_top               -->
+    <!-- Origin: xyz="0 0 1.3", rpy="-1.5708 -1.5708 0"-->
+    <!-- ============================================== -->
+    <joint name="J_F0" type="fixed">
+        <parent link="link_01"/>
+        <child link="link_01_top"/>
+        <origin xyz="0 0 1.3" rpy="-1.5708 -1.5708 0"/>
+    </joint>
+    <!-- ============================================== -->
+    <!-- Link: link_01_top (中间虚拟连杆)               -->
+    <!-- 用于坐标系转换，无实际几何形状                  -->
+    <!-- ============================================== -->
+    <link name="link_01_top">
+        <inertial>
+            <mass value="0.01"/>
+            <origin xyz="0 0 0" rpy="0 0 0"/>
+            <inertia ixx="0.001" ixy="0.0" ixz="0.0" iyy="0.001" iyz="0.0" izz="0.001"/>
+        </inertial>
+    </link>
+    <!-- ============================================== -->
+    <!-- Joint: J_1 (Revolute)                         -->
+    <!-- Connects link_01_top to link_02               -->
+    <!-- Origin: xyz="0 0 0.35", Axis: Z               -->
+    <!-- ============================================== -->
+    <joint name="J_1" type="revolute">
+        <parent link="link_01_top"/>
+        <child link="link_02"/>
+        <origin xyz="0 0 0.35" rpy="0 0 0"/>
+        <axis xyz="0 0 1"/>
+        <limit lower="-3.14" upper="3.14" effort="100" velocity="1.0"/>
+    </joint>
+    <!-- ============================================== -->
+    <!-- Link: link_02 (第二臂/大臂)                    -->
+    <!-- Box: size="0.3 1.2 0.2"                       -->
+    <!-- ============================================== -->
+    <link name="link_02">
+        <visual>
+            <origin xyz="0 0.6 0" rpy="0 0 0"/>
+            <geometry>
+                <box size="0.3 1.2 0.2"/>
+            </geometry>
+            <material name="green"/>
+        </visual>
+        <collision>
+            <origin xyz="0 0.6 0" rpy="0 0 0"/>
+            <geometry>
+                <box size="0.3 1.2 0.2"/>
+            </geometry>
+        </collision>
+        <inertial>
+            <mass value="3.0"/>
+            <origin xyz="0 0.6 0" rpy="0 0 0"/>
+            <inertia ixx="0.3" ixy="0.0" ixz="0.0" iyy="0.3" iyz="0.0" izz="0.3"/>
+        </inertial>
+    </link>
+    <!-- ============================================== -->
+    <!-- Joint: J_2 (Revolute)                         -->
+    <!-- Connects link_02 to link_03                   -->
+    <!-- Origin: xyz="0 0.9 0.2", Axis: Z              -->
+    <!-- ============================================== -->
+    <joint name="J_2" type="revolute">
+        <parent link="link_02"/>
+        <child link="link_03"/>
+        <origin xyz="0 0.9 0.2" rpy="0 0 0"/>
+        <axis xyz="0 0 1"/>
+        <limit lower="-3.14" upper="3.14" effort="100" velocity="1.0"/>
+    </joint>
+    <!-- ============================================== -->
+    <!-- Link: link_03 (第三臂/小臂)                    -->
+    <!-- Box: size="0.2 1.0 0.1"                       -->
+    <!-- ============================================== -->
+    <link name="link_03">
+        <visual>
+            <origin xyz="0 0.5 0" rpy="0 0 0"/>
+            <geometry>
+                <box size="0.2 1.0 0.1"/>
+            </geometry>
+            <material name="orange"/>
+        </visual>
+        <collision>
+            <origin xyz="0 0.5 0" rpy="0 0 0"/>
+            <geometry>
+                <box size="0.2 1.0 0.1"/>
+            </geometry>
+        </collision>
+        <inertial>
+            <mass value="2.0"/>
+            <origin xyz="0 0.5 0" rpy="0 0 0"/>
+            <inertia ixx="0.2" ixy="0.0" ixz="0.0" iyy="0.2" iyz="0.0" izz="0.2"/>
+        </inertial>
+    </link>
+    <!-- ============================================== -->
+    <!-- Joint: J_3 (Revolute)                         -->
+    <!-- Connects link_03 to effector                  -->
+    <!-- Origin: xyz="0 0.9 0.05", rpy="1.5708 1.5708 3.14159" -->
+    <!-- Axis: Z                                       -->
+    <!-- ============================================== -->
+    <joint name="J_3" type="revolute">
+        <parent link="link_03"/>
+        <child link="effector"/>
+        <origin xyz="0 0.9 0.05" rpy="1.5708 1.5708 3.14159"/>
+        <axis xyz="0 0 1"/>
+        <limit lower="-3.14" upper="3.14" effort="100" velocity="1.0"/>
+    </joint>
+    <!-- ============================================== -->
+    <!-- Link: effector (末端执行器)                    -->
+    <!-- Box: size="0.2 0.2 0.1"                       -->
+    <!-- ============================================== -->
+    <link name="effector">
+        <visual>
+            <origin xyz="0 0 0.05" rpy="0 0 0"/>
+            <geometry>
+                <box size="0.2 0.2 0.1"/>
+            </geometry>
+            <material name="red"/>
+        </visual>
+        <collision>
+            <origin xyz="0 0 0.05" rpy="0 0 0"/>
+            <geometry>
+                <box size="0.2 0.2 0.1"/>
+            </geometry>
+        </collision>
+        <inertial>
+            <mass value="0.5"/>
+            <origin xyz="0 0 0.05" rpy="0 0 0"/>
+            <inertia ixx="0.01" ixy="0.0" ixz="0.0" iyy="0.01" iyz="0.0" izz="0.01"/>
+        </inertial>
+    </link>
 </robot>

Commit message: 优化 PUMA 机械臂 URDF 模型，更新材料定义，调整连杆和关节参数，修复几何形状和质量设置

File: src/midterm_model/urdf/robot.urdf.xacro (robot description, xacro)
@@ -2,9 +2,12 @@
 <robot name="puma_robot" xmlns:xacro="http://www.ros.org/wiki/xacro">
     <!-- ============================================== -->
-    <!-- Material Definitions for Visualization        -->
+    <!-- Material Definitions                          -->
     <!-- ============================================== -->
     <material name="blue">
         <color rgba="0.0 0.0 0.8 1.0"/>
     </material>
+    <material name="cyan">
+        <color rgba="0.0 0.8 0.8 1.0"/>
+    </material>
     <material name="green">
         <color rgba="0.0 0.8 0.0 1.0"/>
@@ -15,7 +18,4 @@
     <material name="orange">
         <color rgba="1.0 0.5 0.0 1.0"/>
-    </material>
-    <material name="yellow">
-        <color rgba="1.0 1.0 0.0 1.0"/>
     </material>
     <material name="grey">
@@ -34,4 +34,5 @@
     <!-- Link: base_link (基座)                         -->
     <!-- Cylinder: radius=0.35, length=0.1             -->
+    <!-- Origin: 0 0 0.05                              -->
     <!-- ============================================== -->
     <link name="base_link">
@@ -57,5 +58,4 @@
     <!-- ============================================== -->
     <!-- Joint: J_0 (Revolute)                         -->
-    <!-- Connects base_link to link_01                 -->
     <!-- Origin: xyz="0 0 0.1", Axis: Z                -->
     <!-- ============================================== -->
@@ -68,5 +68,5 @@
     </joint>
     <!-- ============================================== -->
-    <!-- Link: link_01 (第一臂/立柱)                    -->
+    <!-- Link: link_01 (立柱)                           -->
     <!-- Cylinder: radius=0.15, length=1.1             -->
     <!-- ============================================== -->
@@ -92,32 +92,43 @@
     </link>
     <!-- ============================================== -->
-    <!-- Joint: J_F0 (Fixed) - 坐标系转换关节           -->
-    <!-- Connects link_01 to link_01_top               -->
-    <!-- Origin: xyz="0 0 1.3", rpy="-1.5708 -1.5708 0"-->
+    <!-- Joint: J_F0 (Fixed) - 坐标系转换               -->
+    <!-- Origin: xyz="0 0 1.3", rpy="-pi/2 -pi/2 0"    -->
     <!-- ============================================== -->
     <joint name="J_F0" type="fixed">
         <parent link="link_01"/>
-        <child link="link_01_top"/>
+        <child link="link_02"/>
         <origin xyz="0 0 1.3" rpy="-1.5708 -1.5708 0"/>
     </joint>
     <!-- ============================================== -->
-    <!-- Link: link_01_top (中间虚拟连杆)               -->
-    <!-- 用于坐标系转换，无实际几何形状                  -->
-    <!-- ============================================== -->
-    <link name="link_01_top">
-        <inertial>
-            <mass value="0.01"/>
-            <origin xyz="0 0 0" rpy="0 0 0"/>
-            <inertia ixx="0.001" ixy="0.0" ixz="0.0" iyy="0.001" iyz="0.0" izz="0.001"/>
+    <!-- Link: link_02 (水平连接圆柱)                   -->
+    <!-- Cylinder: radius=0.2, length=0.5              -->
+    <!-- ============================================== -->
+    <link name="link_02">
+        <visual>
+            <origin xyz="0 0 0" rpy="0 0 0"/>
+            <geometry>
+                <cylinder radius="0.2" length="0.5"/>
+            </geometry>
+            <material name="cyan"/>
+        </visual>
+        <collision>
+            <origin xyz="0 0 0" rpy="0 0 0"/>
+            <geometry>
+                <cylinder radius="0.2" length="0.5"/>
+            </geometry>
+        </collision>
+        <inertial>
+            <mass value="2.0"/>
+            <origin xyz="0 0 0" rpy="0 0 0"/>
+            <inertia ixx="0.2" ixy="0.0" ixz="0.0" iyy="0.2" iyz="0.0" izz="0.2"/>
         </inertial>
     </link>
     <!-- ============================================== -->
     <!-- Joint: J_1 (Revolute)                         -->
-    <!-- Connects link_01_top to link_02               -->
     <!-- Origin: xyz="0 0 0.35", Axis: Z               -->
     <!-- ============================================== -->
     <joint name="J_1" type="revolute">
-        <parent link="link_01_top"/>
-        <child link="link_02"/>
+        <parent link="link_02"/>
+        <child link="link_03"/>
         <origin xyz="0 0 0.35" rpy="0 0 0"/>
         <axis xyz="0 0 1"/>
@@ -125,10 +136,10 @@
     </joint>
     <!-- ============================================== -->
-    <!-- Link: link_02 (第二臂/大臂)                    -->
+    <!-- Link: link_03 (大臂)                           -->
     <!-- Box: size="0.3 1.2 0.2"                       -->
     <!-- ============================================== -->
-    <link name="link_02">
-        <visual>
-            <origin xyz="0 0.6 0" rpy="0 0 0"/>
+    <link name="link_03">
+        <visual>
+            <origin xyz="0 0.4 0" rpy="0 0 0"/>
             <geometry>
                 <box size="0.3 1.2 0.2"/>
@@ -150,21 +161,20 @@
     <!-- ============================================== -->
     <!-- Joint: J_2 (Revolute)                         -->
-    <!-- Connects link_02 to link_03                   -->
     <!-- Origin: xyz="0 0.9 0.2", Axis: Z              -->
     <!-- ============================================== -->
     <joint name="J_2" type="revolute">
-        <parent link="link_02"/>
-        <child link="link_03"/>
-        <origin xyz="0 0.9 0.2" rpy="0 0 0"/>
-        <axis xyz="0 0 1"/>
-        <limit lower="-3.14" upper="3.14" effort="100" velocity="1.0"/>
-    </joint>
-    <!-- ============================================== -->
-    <!-- Link: link_03 (第三臂/小臂)                    -->
+        <parent link="link_03"/>
+        <child link="link_04"/>
+        <origin xyz="0 0.8 0.2" rpy="0 0 0"/>
+        <axis xyz="0 0 1"/>
+        <limit lower="-3.14" upper="3.14" effort="100" velocity="1.0"/>
+    </joint>
+    <!-- ============================================== -->
+    <!-- Link: link_04 (小臂)                           -->
     <!-- Box: size="0.2 1.0 0.1"                       -->
     <!-- ============================================== -->
-    <link name="link_03">
-        <visual>
-            <origin xyz="0 0.5 0" rpy="0 0 0"/>
+    <link name="link_04">
+        <visual>
+            <origin xyz="0 0.5 -0.05" rpy="0 0 0"/>
             <geometry>
                 <box size="0.2 1.0 0.1"/>
@@ -173,5 +183,5 @@
         </visual>
         <collision>
-            <origin xyz="0 0.5 0" rpy="0 0 0"/>
+            <origin xyz="0 0.5 -0.05" rpy="0 0 0"/>
             <geometry>
                 <box size="0.2 1.0 0.1"/>
@@ -180,5 +190,5 @@
         <inertial>
             <mass value="2.0"/>
-            <origin xyz="0 0.5 0" rpy="0 0 0"/>
+            <origin xyz="0 0.5 -0.05" rpy="0 0 0"/>
             <inertia ixx="0.2" ixy="0.0" ixz="0.0" iyy="0.2" iyz="0.0" izz="0.2"/>
         </inertial>
@@ -186,12 +196,10 @@
     <!-- ============================================== -->
     <!-- Joint: J_3 (Revolute)                         -->
-    <!-- Connects link_03 to effector                  -->
-    <!-- Origin: xyz="0 0.9 0.05", rpy="1.5708 1.5708 3.14159" -->
-    <!-- Axis: Z                                       -->
+    <!-- Origin: xyz="0 0.9 -0.05", rpy="pi/2 pi/2 pi" -->
     <!-- ============================================== -->
     <joint name="J_3" type="revolute">
-        <parent link="link_03"/>
+        <parent link="link_04"/>
         <child link="effector"/>
-        <origin xyz="0 0.9 0.05" rpy="1.5708 1.5708 3.14159"/>
+        <origin xyz="0 1.0 -0.05" rpy="1.5708 1.5708 3.14159"/>
         <axis xyz="0 0 1"/>
         <limit lower="-3.14" upper="3.14" effort="100" velocity="1.0"/>
@@ -210,5 +218,5 @@
         </visual>
         <collision>
-            <origin xyz="0 0 0.05" rpy="0 0 0"/>
+            <origin xyz="0 0 0" rpy="0 0 0"/>
             <geometry>
                 <box size="0.2 0.2 0.1"/>
@@ -217,5 +225,5 @@
         <inertial>
             <mass value="0.5"/>
-            <origin xyz="0 0 0.05" rpy="0 0 0"/>
+            <origin xyz="0 0 0" rpy="0 0 0"/>
             <inertia ixx="0.01" ixy="0.0" ixz="0.0" iyy="0.01" iyz="0.0" izz="0.01"/>
         </inertial>

Commit message: 调整 J_2、J_3 和 effector 关节的原点位置，修正 link_04 的可视化原点，优化 URDF 模型的几何形状

File: src/midterm_model/urdf/robot.urdf.xacro (robot description, xacro)
@@ -161,10 +161,10 @@
     <!-- ============================================== -->
     <!-- Joint: J_2 (Revolute)                         -->
-    <!-- Origin: xyz="0 0.9 0.2", Axis: Z              -->
+    <!-- Origin: xyz="0 1.0 0.2", Axis: Z              -->
     <!-- ============================================== -->
     <joint name="J_2" type="revolute">
         <parent link="link_03"/>
         <child link="link_04"/>
-        <origin xyz="0 0.8 0.2" rpy="0 0 0"/>
+        <origin xyz="0 0.85 0.15" rpy="0 0 0"/>
         <axis xyz="0 0 1"/>
         <limit lower="-3.14" upper="3.14" effort="100" velocity="1.0"/>
@@ -176,5 +176,5 @@
     <link name="link_04">
         <visual>
-            <origin xyz="0 0.5 -0.05" rpy="0 0 0"/>
+            <origin xyz="0 0.4 0" rpy="0 0 0"/>
             <geometry>
                 <box size="0.2 1.0 0.1"/>
@@ -201,5 +201,5 @@
         <parent link="link_04"/>
         <child link="effector"/>
-        <origin xyz="0 1.0 -0.05" rpy="1.5708 1.5708 3.14159"/>
+        <origin xyz="0 1.0 0" rpy="1.5708 1.5708 3.14159"/>
         <axis xyz="0 0 1"/>
         <limit lower="-3.14" upper="3.14" effort="100" velocity="1.0"/>
@@ -211,5 +211,5 @@
     <link name="effector">
         <visual>
-            <origin xyz="0 0 0.05" rpy="0 0 0"/>
+            <origin xyz="-0.0 0 -0.05" rpy="0 0 0"/>
             <geometry>
                 <box size="0.2 0.2 0.1"/>
